Commit message: Created drivers and new working gazebo model

File: urdf/ezrassor.xacro (robot description, xacro)
@@ -176,8 +176,4 @@
       <mass value="5"/>
       <xacro:cylinder_inertia m="5" r="0.05" h="0.3"/>
-      <inertia
-        ixx="1.0" ixy="0.0" ixz="0.0"
-        iyy="1.0" iyz="0.0"
-        izz="1.0"/>
     </inertial>
   </link>
@@ -232,87 +228,4 @@
     </inertial>
   </link>
-  <!-- Transmissions -->
-  <!--
-  <transmission name="left_wheel_front_tran">
-    <type>transmission_interface/SimpleTransmission</type>
-    <joint name="left_wheel_front_hinge">
-      <hardwareInterface>hardware_interface/VelocityJointInterface</hardwareInterface>
-    </joint>
-    <actuator name="left_wheel_front_motor">
-      <hardwareInterface>hardware_interface/VelocityJointInterface</hardwareInterface>
-      <mechanicalReduction>1</mechanicalReduction>
-    </actuator>
-  </transmission>
-  <transmission name="left_wheel_back_tran">
-    <type>transmission_interface/SimpleTransmission</type>
-    <joint name="left_wheel_back_hinge">
-      <hardwareInterface>hardware_interface/VelocityJointInterface</hardwareInterface>
-    </joint>
-    <actuator name="left_wheel_back_motor">
-      <hardwareInterface>hardware_interface/VelocityJointInterface</hardwareInterface>
-      <mechanicalReduction>1</mechanicalReduction>
-    </actuator>
-  </transmission>
-  <transmission name="right_wheel_front_tran">
-    <type>transmission_interface/SimpleTransmission</type>
-    <joint name="right_wheel_front_hinge">
-      <hardwareInterface>hardware_interface/VelocityJointInterface</hardwareInterface>
-    </joint>
-    <actuator name="right_wheel_front_motor">
-      <hardwareInterface>hardware_interface/VelocityJointInterface</hardwareInterface>
-      <mechanicalReduction>1</mechanicalReduction>
-    </actuator>
-  </transmission>
-  <transmission name="right_wheel_back_tran">
-    <type>transmission_interface/SimpleTransmission</type>
-    <joint name="right_wheel_back_hinge">
-      <hardwareInterface>hardware_interface/VelocityJointInterface</hardwareInterface>
-    </joint>
-    <actuator name="right_wheel_back_motor">
-      <hardwareInterface>hardware_interface/VelocityJointInterface</hardwareInterface>
-      <mechanicalReduction>1</mechanicalReduction>
-    </actuator>
-  </transmission>
-  <transmission name="arm_front_tran">
-    <type>transmission_interface/SimpleTransmission</type>
-    <joint name="arm_front_hinge">
-      <hardwareInterface>hardware_interface/VelocityJointInterface</hardwareInterface>
-    </joint>
-    <actuator name="arm_front_motor">
-      <hardwareInterface>hardware_interface/VelocityJointInterface</hardwareInterface>
-      <mechanicalReduction>1</mechanicalReduction>
-    </actuator>
-  </transmission>
-  <transmission name="arm_back_tran">
-    <type>transmission_interface/SimpleTransmission</type>
-    <joint name="arm_back_hinge">
-      <hardwareInterface>hardware_interface/VelocityJointInterface</hardwareInterface>
-    </joint>
-    <actuator name="arm_back_motor">
-      <hardwareInterface>hardware_interface/VelocityJointInterface</hardwareInterface>
-      <mechanicalReduction>1</mechanicalReduction>
-    </actuator>
-  </transmission>
-  <transmission name="drum_front_hinge_tran">
-    <type>transmission_interface/SimpleTransmission</type>
-    <joint name="drum_front_hinge">
-      <hardwareInterface>hardware_interface/VelocityJointInterface</hardwareInterface>
-    </joint>
-    <actuator name="drum_front_hinge_motor">
-      <hardwareInterface>hardware_interface/VelocityJointInterface</hardwareInterface>
-      <mechanicalReduction>1</mechanicalReduction>
-    </actuator>
-  </transmission>
-  <transmission name="drum_back_hinge_tran">
-    <type>transmission_interface/SimpleTransmission</type>
-    <joint name="drum_back_hinge">
-      <hardwareInterface>hardware_interface/VelocityJointInterface</hardwareInterface>
-    </joint>
-    <actuator name="drum_back_hinge_motor">
-      <hardwareInterface>hardware_interface/VelocityJointInterface</hardwareInterface>
-      <mechanicalReduction>1</mechanicalReduction>
-    </actuator>
-  </transmission>
-  -->
   <!-- Front Camera Added -->
   <link name="depth_camera_front">
@@ -448,78 +361,77 @@
   <!-- ros2_control configuration for each joint to be used with Gazebo_ros2_control-->
   <ros2_control name="GazeboSystem" type="system">
-            <hardware>
-                <plugin>gazebo_ros2_control/GazeboSystem</plugin>
-            </hardware>
-            <joint name="left_wheel_front_joint">
-            <command_interface name="velocity">
-                <param name="min">-10</param>
-                <param name="max">10</param>
-            </command_interface>
-            <state_interface name="position" />
-            <state_interface name="velocity" />
-        </joint>
-        <joint name="left_wheel_back_joint">
-            <command_interface name="velocity">
-                <param name="min">-10</param>
-                <param name="max">10</param>
-            </command_interface>
-            <state_interface name="position" />
-            <state_interface name="velocity" />
-        </joint>
-        <joint name="right_wheel_front_joint">
-            <command_interface name="velocity">
-                <param name="min">-10</param>
-                <param name="max">10</param>
-            </command_interface>
-            <state_interface name="position" />
-            <state_interface name="velocity" />
-        </joint>
-        <joint name="right_wheel_back_joint">
-            <command_interface name="velocity">
-                <param name="min">-10</param>
-                <param name="max">10</param>
-            </command_interface>
-            <state_interface name="position" />
-            <state_interface name="velocity" />
-        </joint>
-        <joint name="arm_back_joint">
-            <command_interface name="velocity">
-                <param name="min">-10</param>
-                <param name="max">10</param>
-            </command_interface>
-            <state_interface name="position" />
-            <state_interface name="velocity" />
-        </joint>
-        <joint name="drum_back_joint">
-            <command_interface name="velocity">
-                <param name="min">-10</param>
-                <param name="max">10</param>
-            </command_interface>
-            <state_interface name="position" />
-            <state_interface name="velocity" />
-        </joint>
-        <joint name="arm_front_joint">
-            <command_interface name="velocity">
-                <param name="min">-10</param>
-                <param name="max">10</param>
-            </command_interface>
-            <state_interface name="position" />
-            <state_interface name="velocity" />
-        </joint>
-        <joint name="drum_front_joint">
-            <command_interface name="velocity">
-                <param name="min">-10</param>
-                <param name="max">10</param>
-            </command_interface>
-            <state_interface name="position" />
-            <state_interface name="velocity" />
-        </joint>
-        </ros2_control>
-  <!-- Include the gazebo_ros2_control plugin with standard rover model controllers-->
+    <hardware>
+      <plugin>gazebo_ros2_control/GazeboSystem</plugin>
+    </hardware>
+    <joint name="left_wheel_front_joint">
+      <command_interface name="velocity">
+        <param name="min">-1</param>
+        <param name="max">1</param>
+      </command_interface>
+      <state_interface name="position"/>
+      <state_interface name="velocity"/>
+    </joint>
+    <joint name="right_wheel_front_joint">
+      <command_interface name="velocity">
+        <param name="min">-1</param>
+        <param name="max">1</param>
+      </command_interface>
+      <state_interface name="position"/>
+      <state_interface name="velocity"/>
+    </joint>
+    <joint name="left_wheel_back_joint">
+      <command_interface name="velocity">
+        <param name="min">-1</param>
+        <param name="max">1</param>
+      </command_interface>
+      <state_interface name="position"/>
+      <state_interface name="velocity"/>
+    </joint>
+    <joint name="right_wheel_back_joint">
+      <command_interface name="velocity">
+        <param name="min">-1</param>
+        <param name="max">1</param>
+      </command_interface>
+      <state_interface name="position"/>
+      <state_interface name="velocity"/>
+    </joint>
+    <joint name="arm_front_joint">
+      <command_interface name="velocity">
+        <param name="min">-1</param>
+        <param name="max">1</param>
+      </command_interface>
+      <state_interface name="position"/>
+      <state_interface name="velocity"/>
+    </joint>
+    <joint name="arm_back_joint">
+      <command_interface name="velocity">
+        <param name="min">-1</param>
+        <param name="max">1</param>
+      </command_interface>
+      <state_interface name="position"/>
+      <state_interface name="velocity"/>
+    </joint>
+    <joint name="drum_front_joint">
+      <command_interface name="velocity">
+        <param name="min">-1</param>
+        <param name="max">1</param>
+      </command_interface>
+      <state_interface name="position"/>
+      <state_interface name="velocity"/>
+    </joint>
+    <joint name="drum_back_joint">
+      <command_interface name="velocity">
+        <param name="min">-1</param>
+        <param name="max">1</param>
+      </command_interface>
+      <state_interface name="position"/>
+      <state_interface name="velocity"/>
+    </joint>
+  </ros2_control>
   <gazebo>
-    <plugin filename="libgazebo_ros2_control.so" name="gazebo_ros2_control">
-      <parameters>$(find ezrassor_robot_description)/config/standard_rover/default_position_controllers.yaml</parameters>
-    </plugin>
-  </gazebo>
-  <plugin filename="libgazebo_ros_state.so" name="gazebo_ros_state"/>
+        <!-- Joint state publisher -->
+        <plugin filename="libgazebo_ros2_control.so" name="gazebo_ros2_control">
+            <parameters>$(find ezrassor_robot_description)/config/ezrassor_basic_controllers.yaml</parameters>
+        </plugin>
+    </gazebo>
 </robot>

File: urdf/ezrassor_rviz.xacro (robot description, xacro)
@@ -3,5 +3,4 @@
   <xacro:property name="cameraSize" value="0.01"/>
   <xacro:property name="cameraMass" value="0.1"/>
-  <xacro:include filename="$(find ezrassor_robot_description)/urdf/ezrassor.gazebo" />
   <xacro:include filename="$(find ezrassor_robot_description)/urdf/materials.xacro" />
   <xacro:include filename="$(find ezrassor_robot_description)/urdf/macros.xacro" />
@@ -13,5 +12,5 @@
     <pose>0 0 0 0 0 0</pose>
     <inertial>
-      <mass value="15.0"/>
+      <mass value="1.5"/>
       <origin xyz="0 0 0" rpy=" 0 0 0"/>
       <inertia
@@ -61,6 +60,6 @@
     <inertial>
       <origin xyz="0 0 0" rpy="0 0 0" />
-      <mass value="5"/>
-      <xacro:cylinder_inertia m="5" r="0.18" h="0.2"/>
+      <mass value="0.5"/>
+      <xacro:cylinder_inertia m="0.5" r="0.18" h="0.2"/>
     </inertial>
   </link>
@@ -86,6 +85,6 @@
     <inertial>
       <origin xyz="0 0 0" rpy="0 0 3.14159"/>
-      <mass value="5"/>
-      <xacro:cylinder_inertia m="5" r="0.18" h="0.2"/>
+      <mass value="0.5"/>
+      <xacro:cylinder_inertia m="0.5" r="0.18" h="0.2"/>
     </inertial>
   </link>
@@ -111,6 +110,6 @@
     <inertial>
       <origin xyz="0 0 0" rpy="0 0 0"/>
-      <mass value="5"/>
-      <xacro:cylinder_inertia m="5" r="0.18" h="0.2"/>
+      <mass value="0.5"/>
+      <xacro:cylinder_inertia m="0.5" r="0.18" h="0.2"/>
     </inertial>
   </link>
@@ -136,6 +135,6 @@
     <inertial>
       <origin xyz="0 0 0" rpy="0 0 3.14159"/>
-      <mass value="5"/>
-      <xacro:cylinder_inertia m="5" r="0.18" h="0.2"/>
+      <mass value="0.5"/>
+      <xacro:cylinder_inertia m="0.5" r="0.18" h="0.2"/>
     </inertial>
   </link>
@@ -155,6 +154,6 @@
     <inertial>
       <origin xyz="0 0 0" rpy="0 0 0"/>
-      <mass value="5"/>
-      <xacro:cylinder_inertia m="5" r="0.05" h="0.3"/>
+      <mass value="0.5"/>
+      <xacro:cylinder_inertia m="0.5" r="0.05" h="0.3"/>
     </inertial>
   </link>
@@ -174,6 +173,6 @@
     <inertial>
       <origin xyz="0 0 0" rpy="0 0 3.1415"/>
-      <mass value="5"/>
-      <xacro:cylinder_inertia m="5" r="0.05" h="0.3"/>
+      <mass value="0.5"/>
+      <xacro:cylinder_inertia m="0.5" r="0.05" h="0.3"/>
       <inertia
         ixx="1.0" ixy="0.0" ixz="0.0"
@@ -203,6 +202,6 @@
     <inertial>
       <origin xyz="0 0 0" rpy="0 0 0"/>
-      <mass value="5"/>
-      <xacro:cylinder_inertia m="5" r="0.1839" h="1.0"/>
+      <mass value="0.5"/>
+      <xacro:cylinder_inertia m="0.5" r="0.1839" h="1.0"/>
     </inertial>
   </link>
@@ -228,6 +227,6 @@
     <inertial>
       <origin xyz="0 0 0" rpy="0 0 3.14159"/>
-      <mass value="5"/>
-      <xacro:cylinder_inertia m="5" r="0.1839" h="1.0"/>
+      <mass value="0.5"/>
+      <xacro:cylinder_inertia m="0.5" r="0.1839" h="1.0"/>
     </inertial>
   </link>
@@ -388,5 +387,5 @@
     <axis xyz="0 1 0" rpy="0 0 0"/>
     <limit effort="100" velocity="100"/>
-    <joint_properties damping="0.0" friction="0.0"/>
+    <joint_properties damping="0.0" friction="1.0"/>
   </joint>
   <joint type="continuous" name="right_wheel_front_joint">
@@ -396,5 +395,5 @@
     <axis xyz="0 1 0" rpy="0 0 0"/>
     <limit effort="100" velocity="100"/>
-    <joint_properties damping="0.0" friction="0.0"/>
+    <joint_properties damping="0.0" friction="1.0"/>
   </joint>
   <joint type="continuous" name="left_wheel_back_joint">
@@ -404,5 +403,5 @@
     <axis xyz="0 1 0" rpy="0 0 0"/>
     <limit effort="100" velocity="100"/>
-    <joint_properties damping="0.0" friction="0.0"/>
+    <joint_properties damping="0.0" friction="1.0"/>
   </joint>
   <joint type="continuous" name="right_wheel_back_joint">
@@ -412,5 +411,5 @@
     <axis xyz="0 1 0" rpy="0 0 0"/>
     <limit effort="100" velocity="100"/>
-    <joint_properties damping="0.0" friction="0.0"/>
+    <joint_properties damping="0.0" friction="1.0"/>
   </joint>
   <joint type="continuous" name="arm_front_joint">

File: urdf/macros.xacro (robot description, xacro)
@@ -40,14 +40,17 @@
     </xacro:macro>
     <xacro:macro name="robot_arm_drum">
-        <mesh filename="package://ezrassor_robot_description/meshes/drum.dae" scale="0.35 0.35 0.35"></mesh>
+        <mesh filename="$(find ezrassor_robot_description)/meshes/drum.dae" scale="0.35 0.35 0.35"></mesh>
     </xacro:macro>
     <xacro:macro name="robot_wheel">
-        <mesh filename="package://ezrassor_robot_description/meshes/wheel.dae" scale="0.35 0.35 0.35"></mesh>
+        <mesh filename="$(find ezrassor_robot_description)/meshes/wheel.dae" scale="0.35 0.35 0.35"></mesh>
     </xacro:macro>
     <xacro:macro name="base_unit">
-        <mesh filename="package://ezrassor_robot_description/meshes/base_unit.dae" scale="0.35 0.35 0.35"></mesh>
+        <!--
+            <mesh filename="package://ezrassor_robot_description/meshes/base_unit.dae" scale="0.35 0.35 0.35"></mesh>
+        -->
+        <mesh filename="$(find ezrassor_robot_description)/meshes/base_unit.dae" scale="0.35 0.35 0.35"></mesh>
     </xacro:macro>
-    <xacro:macro name="drum_arm">
-        <mesh filename="package://ezrassor_robot_description/meshes/drum_arm.dae" scale="0.35 0.35 0.35"></mesh>
+    <xacro:macro name="drum_arm_mesh">
+        <mesh filename="$(find ezrassor_robot_description)/meshes/drum_arm.dae" scale="0.35 0.35 0.35"></mesh>
     </xacro:macro>
     <!-- ARM VISUAL AND COLLISION MACROS -->
