Commit message: Changed drum arm to effort controller

File: urdf/drum_arm.xacro (robot description, xacro)
@@ -41,5 +41,5 @@
             </inertial>
         </link>
-        <joint type="continuous" name="arm_${pos}_joint">
+        <joint type="revolute" name="arm_${pos}_joint">
             <xacro:if value='${pos == "front"}'>
                 <origin xyz="0.20 0 0" rpy="3.1415 0 0"/>
@@ -51,5 +51,5 @@
             <parent link="base_link"/>
             <axis xyz="0 1 0" rpy="0 0 0"/>
-            <limit effort="100" velocity="100"/>
+            <limit effort="1000.0" lower="0" upper="0.71" velocity="0.2"/>
             <joint_properties damping="0.0" friction="0.0"/>
         </joint>

File: urdf/ezrassor_basic.xacro (robot description, xacro)
@@ -92,4 +92,23 @@
         </joint>
         <joint name="arm_front_joint">
+            <command_interface name="effort">
+                <param name="min">-100</param>
+                <param name="max">100</param>
+            </command_interface>
+            <state_interface name="velocity"/>
+            <state_interface name="position"/>
+            <state_interface name="effort"/>
+        </joint>
+        <joint name="arm_back_joint">
+            <command_interface name="effort">
+                <param name="min">-100</param>
+                <param name="max">100</param>
+            </command_interface>
+            <state_interface name="velocity"/>
+            <state_interface name="position"/>
+            <state_interface name="effort"/>
+        </joint>
+        <!--
+        <joint name="arm_front_joint">
             <command_interface name="velocity">
                 <param name="min">-1</param>
@@ -107,4 +126,5 @@
             <state_interface name="position"/>
         </joint>
+        -->
         <joint name="drum_front_joint">
             <command_interface name="velocity">
